Commit message: Changed path planner and moved robot closer to objects

File: conveyer-belt-cv-package/models/camera/model.urdf (robot description, URDF)
Before this commit: robot None, 2 links, 1 joints
Links:
- link camera_link: geometry collision box size=0.1 0.1 0.1; visual box size=0.1 0.1 0.1
